File: bldc_servo_driver_mini_G4/sch/int_sensor/bldc_servo_driver_mini_i.kicad_pcb (KiCad board)
At the start: 4 copper layers, 35.5 x 34.7 mm, 71 parts, among them IC1 ST730MR, IC2 LT1616ES6#TRMPBF, IC3 TLT9251VLEXUMA1, IC4 STM32G491CCU6, J1 1-2328702-0, J2 Conn_01x04, J3 Conn_01x04, J7 DF65-3P-1.7V_21_, U1 AS5048A, U2 PDRV8311HRRWR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

Commit message: fix : bldc servo driver mini sch
Parts:
- added TP1: TestPoint, TestPoint:TestPoint_Pad_D1.0mm, F.Cu at (117.6, 72.8)
- added TP2: TestPoint, TestPoint:TestPoint_Pad_D1.0mm, F.Cu at (130.8, 75.8)
- added TP3: TestPoint, TestPoint:TestPoint_Pad_D1.0mm, F.Cu at (132.6, 75.8)
- IC4: value STM32G491CCU6 -> STM32G4xxyU
- R19: value 30.1k -> 30.1k or 51k(MP2359)
Routing:
- net /Potentio_Sens: track 0.00 -> 5.01 mm, vias 0 -> 2
- net GND: track 14.3 -> 17.3 mm, vias 63 -> 59
- net +3V3: track 107.1 -> 108.6 mm
- net /NRST: track 31.8 -> 31.3 mm
Other:
- board text added: "FMSKF ServoDriverMini V2cc"
- board text removed: "FMSKF ServoDriverMini V1cc"
